File: zynqPCB/LCD50.kicad_sch (KiCad schematic)
At the start: 29 parts, among them J4 HDMI_A, Q2 IRLML2502, Q3 IRLML2502, Q4 IRLML2502, U19 PCA9306, U20B1 xc7z020clg484, U20D1 xc7z020clg484, U20E1 xc7z020clg484

Commit message: Sensores Removed
Connections:
- net ACC_INT1: no longer names the net of U20B1.W12 (IO_L4N_T0_13)
- net ACC_INT2: no longer names the net of U20B1.V12 (IO_L4P_T0_13)
- net RF_IRQ: no longer names the net of U20B1.AA11 (IO_L8P_T1_13)
- net TEMPO_LED: no longer names the net of U20B1.R6 (IO_L19P_T3_13)
- no-connect marks 19 -> 24
Changed lines of the file:
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@@
+	)
+	(no_connect
+		(at 160.02 88.9)
 	)
 	(no_connect
@@
 	)
 	(no_connect
+		(at 163.83 64.77)
+	)
+	(no_connect
+		(at 163.83 87.63)
+	)
+	(no_connect
 		(at 163.83 59.69)
 	)
@@
 	(no_connect
 		(at 163.83 54.61)
+	)
+	(no_connect
+		(at 163.83 67.31)
+	)
+	(no_connect
+		(at 163.83 143.51)
 	)
 	(wire
@@
 		)
 	)
-	(global_label "ACC_INT2"
-		(shape bidirectional)
-		(at 163.83 67.31 180)
-		(effects
-			(font
-				(size 1.524 1.524)
-			)
-			(justify right)
-		)
-		(property "Intersheetrefs" "${INTERSHEET_REFS}"
-			(at 163.83 67.31 0)
-			(effects
-				(font
-					(size 1.27 1.27)
-				)
-				(hide yes)
-			)
-		)
-	)
 	(global_label "STATLED_2"
 		(shape output)
@@
 		)
 	)
-	(global_label "RF_IRQ"
-		(shape bidirectional)
-		(at 163.83 87.63 180)
-		(effects
-			(font
-				(size 1.524 1.524)
-			)
-			(justify right)
-		)
-		(property "Intersheetrefs" "${INTERSHEET_REFS}"
-			(at 163.83 87.63 0)
-			(effects
-				(font
-					(size 1.27 1.27)
-				)
-				(hide yes)
-			)
-		)
-	)
 	(global_label "LCD_D2"
 		(shape bidirectional)
@@
 		)
 	)
-	(global_label "ACC_INT1"
-		(shape bidirectional)
-		(at 163.83 64.77 180)
-		(effects
-			(font
-				(size 1.524 1.524)
-			)
-			(justify right)
-		)
-		(property "Intersheetrefs" "${INTERSHEET_REFS}"
-			(at 163.83 64.77 0)
-			(effects
-				(font
-					(size 1.27 1.27)
-				)
-				(hide yes)
-			)
-		)
-	)
 	(global_label "LCD_D8"
 		(shape bidirectional)
@@
 			(effects
 				(font
-					(size 1.27 1.27)
-				)
-				(hide yes)
-			)
-		)
-	)
-	(global_label "TEMPO_LED"
-		(shape output)
-		(at 163.83 143.51 180)
-		(effects
-			(font
-				(size 1.524 1.524)
-			)
-			(justify right)
-		)
-		(property "Intersheetrefs" "${INTERSHEET_REFS}"
-			(at 163.83 143.51 0)
-			(effects
-				(font

Commit message: sensor changed
Parts:
- added R103, R104, R105: R, symbol DFTCustom:R
Connections:
- net GND: now also R103.1, R104.1, R105.1
- net at U20B1.AA11 (IO_L8P_T1_13): now also R105.2
- net TEMPO_LED: now reaches U20B1.R6 (IO_L19P_T3_13)
- net at U20B1.V12 (IO_L4P_T0_13): now also R104.2
- net at U20B1.W12 (IO_L4N_T0_13): now also R103.2
- no-connect marks 24 -> 19
