File: zynqPCB/Storage.kicad_sch (KiCad schematic)
At the start: 22 parts, among them J3 Micro_SD_Card_Det, U16 FTDITypeUART, U17 ABRACON-ASDMB, U18 S25FL256SAGNFI001, U20F1 xc7z020clg484

Commit message: Cleared ERC error except the sequencer Part
Parts:
- added C10: .47uF, Capacitor_SMD:C_0402_1005Metric, symbol Device:C_Small
- added C11: 4.7uF, Capacitor_SMD:C_0402_1005Metric, symbol Device:C_Small
- added C12: 100uF, Capacitor_SMD:C_1210_3225Metric, symbol Device:C_Small
- added R7: 10k, Resistor_SMD:R_0402_1005Metric, symbol Device:R
- added R8: 47, Resistor_SMD:R_0402_1005Metric, symbol Device:R_Small
- added unit 7 of U20
- renumbered U20F1 to U20
Connections:
- net +3.3V: now also C10.1, C11.1, C12.1, R7.2, U20.A10 (VCCO_MIO1_501[4]), U20.B13 (VCCO_MIO1_501[4]), U20.D9 (VCCO_MIO1_501[4]), U20.E12 (VCCO_MIO1_501[4])
- net GND: now also C10.2, C11.2, C12.2
- net SD_CD: now also U20.A13 (PS_MIO26_501)
- net SD_CLK: now also R8.2
- net SD_CMD: now also U20.E9 (PS_MIO17_501)
- net SD_D0: now also U20.A7 (PS_MIO18_501)
- net SD_D1: now also U20.E10 (PS_MIO19_501)
- net SD_D2: now also U20.A8 (PS_MIO20_501)
- net SD_D3: now also U20.F11 (PS_MIO21_501)
- new net: R7.1, U20.C9 (PS_SRST_B_501)
- new net: R8.1, U20.D6 (PS_MIO16_501)
- no-connect marks 6 -> 37
Other:
- moved on the sheet: C89, C90, C91, C92, J3, R63, R64, R65, R66, R67, R68, R69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
