File: zynqPCB/DDR3.kicad_sch (KiCad schematic)
At the start: 62 parts, among them U15 TPS51200DRCR, U20H1 xc7z020clg484, U24 MT41K256M16TW-107_P, U25 MT41K256M16TW-107_P

Commit message: Cleared ERC error except the sequencer Part
Parts:
- renumbered U20H1 to U20
Changed lines of the file:
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@@
 		(in_pos_files yes)
 		(dnp no)
-		(property "Reference" "U20H1"
+		(property "Reference" "U20"
 			(at 289.0774 105.3338 0)
 			(show_name no)
@@
 			(project "DFTBoard"
 				(path "/49eba173-d38c-4d05-b21c-b4a14c4948c2/00000000-0000-0000-0000-000058818a06"
-					(reference "U20H1")
+					(reference "U20")
 					(unit 8)
 				)

Commit message: Sanity Checks and added some footprints
Parts:
- U24, U25: footprint MT41K256M16TW-107_P:BGA96C80P9X16_1400X800X120 -> DFTcustom:MT41K256M16TW_107_P
Changed lines of the file:
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@@
 			)
 		)
-		(property "Footprint" "MT41K256M16TW-107_P:BGA96C80P9X16_1400X800X120"
+		(property "Footprint" "DFTcustom:MT41K256M16TW_107_P"
 			(at 123.19 88.9 0)
 			(hide yes)
@@
 			)
 		)
-		(property "Footprint" "MT41K256M16TW-107_P:BGA96C80P9X16_1400X800X120"
+		(property "Footprint" "DFTcustom:MT41K256M16TW_107_P"
 			(at 27.94 88.9 0)
 			(hide yes)
